File: Linkable_LED_Matrix PCB/Linkable_LED_Matrix_Thru_Full_Mount.sch (EAGLE design)
At the start: 9 parts, among them J1 AVR_SPI_PRG_6NS

Commit message: Fixed silk screen and shifted JP2 very slightly
Parts:
- removed J1: AVR_SPI_PRG_6NS, SparkFun-Connectors:AVR_SPI_PRG_6NS
- removed JP1, JP2: (no value), pinhead:PINHD-1X6
- added U$6, U$7: DIP1X6MALE, ScottSilver:DIP1X6MALE
- added U$9: DIP2X3MALE, ScottSilver:DIP2X3MALE
Connections:
- net CS: now also U$6.3, U$7.3; no longer JP1.4, JP2.4
- net GND: now also U$6.1, U$7.1, U$9.GND; no longer J1.6, JP1.6, JP2.6
- net MISO: now also U$7.4, U$9.MISO; no longer J1.1, JP2.3
- net MOSI: now also U$6.4, U$9.MOSI; no longer J1.4, JP1.3
- net RESET: now also U$6.2, U$7.2, U$9.RESET; no longer J1.5, JP1.5, JP2.5
- net SCK: now also U$6.5, U$7.5, U$9.SCK; no longer J1.3, JP1.2, JP2.2
- net VCC: now also U$6.6, U$7.6, U$9.+5; no longer J1.2, JP1.1, JP2.1
Changed lines of the file:
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@@
 <part name="SUPPLY5" library="SparkFun-Aesthetics" deviceset="VCC" device=""/>
 <part name="GND5" library="SparkFun-Aesthetics" deviceset="GND" device=""/>
-<part name="J1" library="SparkFun-Connectors" deviceset="AVR_SPI_PRG_6" device="NS"/>
 <part name="GND6" library="SparkFun-Aesthetics" deviceset="GND" device=""/>
 <part name="SUPPLY6" library="SparkFun-Aesthetics" deviceset="VCC" device=""/>
 <part name="R1" library="resistor" deviceset="R-US_" device="R0603"/>
-<part name="JP1" library="pinhead" deviceset="PINHD-1X6" device=""/>
-<part name="JP2" library="pinhead" deviceset="PINHD-1X6" device=""/>
 <part name="U$5" library="ScottSilver" deviceset="1X1MM_PAD" device=""/>
+<part name="U$6" library="ScottSilver" deviceset="DIP1X6MALE" device=""/>
+<part name="U$7" library="ScottSilver" deviceset="DIP1X6MALE" device=""/>
+<part name="U$9" library="ScottSilver" deviceset="DIP2X3MALE" device=""/>
 </parts>
 <sheets>
@@
 <instance part="SUPPLY5" gate="G$1" x="142.24" y="144.78"/>
 <instance part="GND5" gate="1" x="142.24" y="114.3"/>
-<instance part="J1" gate="G$1" x="22.86" y="78.74"/>
 <instance part="GND6" gate="1" x="40.64" y="73.66"/>
 <instance part="SUPPLY6" gate="G$1" x="40.64" y="81.28"/>
 <instance part="R1" gate="G$1" x="-5.08" y="160.02"/>
-<instance part="JP1" gate="A" x="-17.78" y="142.24" rot="MR0"/>
-<instance part="JP2" gate="A" x="152.4" y="129.54"/>
 <instance part="U$5" gate="G$1" x="30.48" y="119.38" rot="R180"/>
+<instance part="U$6" gate="G$1" x="-15.24" y="142.24"/>
+<instance part="U$7" gate="G$1" x="149.86" y="129.54"/>
+<instance part="U$9" gate="G$1" x="17.78" y="78.74"/>
 </instances>
 <busses>
@@
 <pinref part="R1" gate="G$1" pin="1"/>
 <wire x1="-10.16" y1="160.02" x2="-10.16" y2="162.56" width="0.1524" layer="91"/>
-<pinref part="JP1" gate="A" pin="1"/>
 <wire x1="-10.16" y1="160.02" x2="-10.16" y2="149.86" width="0.1524" layer="91"/>
-<wire x1="-10.16" y1="149.86" x2="-15.24" y2="149.86" width="0.1524" layer="91"/>
+<pinref part="U$6" gate="G$1" pin="6"/>
+<wire x1="-15.24" y1="149.86" x2="-10.16" y2="149.86" width="0.1524" layer="91"/>
 </segment>
 <segment>
 <pinref part="SUPPLY6" gate="G$1" pin="VCC"/>
-<pinref part="J1" gate="G$1" pin="2"/>
 <wire x1="40.64" y1="81.28" x2="33.02" y2="81.28" width="0.1524" layer="91"/>
+<pinref part="U$9" gate="G$1" pin="+5"/>
 </segment>
 <segment>
 <pinref part="SUPPLY5" gate="G$1" pin="VCC"/>
-<pinref part="JP2" gate="A" pin="1"/>
 <wire x1="142.24" y1="144.78" x2="142.24" y2="137.16" width="0.1524" layer="91"/>
 <wire x1="142.24" y1="137.16" x2="149.86" y2="137.16" width="0.1524" layer="91"/>
+<pinref part="U$7" gate="G$1" pin="6"/>
 </segment>
 </net>
@@
 </segment>
 <segment>
-<pinref part="J1" gate="G$1" pin="6"/>
 <pinref part="GND6" gate="1" pin="GND"/>
 <wire x1="33.02" y1="76.2" x2="40.64" y2="76.2" width="0.1524" layer="91"/>
+<pinref part="U$9" gate="G$1" pin="GND"/>
 </segment>
 <segment>
 <pinref part="GND5" gate="1" pin="GND"/>
-<pinref part="JP2" gate="A" pin="6"/>
 <wire x1="142.24" y1="116.84" x2="142.24" y2="124.46" width="0.1524" layer="91"/>
 <wire x1="142.24" y1="124.46" x2="149.86" y2="124.46" width="0.1524" layer="91"/>
+<pinref part="U$7" gate="G$1" pin="1"/>
 </segment>
 <segment>
 <pinref part="GND4" gate="1" pin="GND"/>
-<pinref part="JP1" gate="A" pin="6"/>
 <wire x1="-10.16" y1="127" x2="-10.16" y2="137.16" width="0.1524" layer="91"/>
-<wire x1="-10.16" y1="137.16" x2="-15.24" y2="137.16" width="0.1524" layer="91"/>
+<pinref part="U$6" gate="G$1" pin="1"/>
+<wire x1="-15.24" y1="137.16" x2="-10.16" y2="137.16" width="0.1524" layer="91"/>
 </segment>
 </net>
@@
 </segment>
 <segment>
-<pinref part="J1" gate="G$1" pin="3"/>
-<wire x1="15.24" y1="78.74" x2="10.16" y2="78.74" width="0.1524" layer="91"/>
-<label x="10.16" y="78.74" size="0.8128" layer="95" rot="R180" xref="yes"/>
-</segment>
-<segment>
-<pinref part="JP1" gate="A" pin="2"/>
+<wire x1="149.86" y1="134.62" x2="134.62" y2="134.62" width="0.1524" layer="91"/>
+<label x="134.62" y="134.62" size="1.016" layer="95" rot="R180" xref="yes"/>
+<pinref part="U$7" gate="G$1" pin="5"/>
+</segment>
+<segment>
+<pinref part="U$6" gate="G$1" pin="5"/>
 <wire x1="-15.24" y1="147.32" x2="0" y2="147.32" width="0.1524" layer="91"/>
 <label x="0" y="147.32" size="1.016" layer="95" xref="yes"/>
 </segment>
 <segment>
-<pinref part="JP2" gate="A" pin="2"/>
-<wire x1="149.86" y1="134.62" x2="134.62" y2="134.62" width="0.1524" layer="91"/>
-<label x="134.62" y="134.62" size="1.016" layer="95" rot="R180" xref="yes"/>
+<pinref part="U$9" gate="G$1" pin="SCK"/>
+<wire x1="10.16" y1="78.74" x2="2.54" y2="78.74" width="0.1524" layer="91"/>
+<label x="2.54" y="78.74" size="1.016" layer="95" rot="R180" xref="yes"/>
 </segment>
 </net>
@@
 </segment>
 <segment>
-<pinref part="J1" gate="G$1" pin="1"/>
-<wire x1="15.24" y1="81.28" x2="10.16" y2="81.28" width="0.1524" layer="91"/>
-<label x="10.16" y="81.28" size="0.8128" layer="95" rot="R180" xref="yes"/>
-</segment>
-<segment>
-<pinref part="JP2" gate="A" pin="3"/>
 <wire x1="149.86" y1="132.08" x2="134.62" y2="132.08" width="0.1524" layer="91"/>
 <label x="134.62" y="132.08" size="1.016" layer="95" rot="R180" xref="yes"/>
+<pinref part="U$7" gate="G$1" pin="4"/>
+</segment>
+<segment>
+<pinref part="U$9" gate="G$1" pin="MISO"/>
+<wire x1="10.16" y1="81.28" x2="2.54" y2="81.28" width="0.1524" layer="91"/>
+<label x="2.54" y="81.28" size="1.016" layer="95" rot="R180" xref="yes"/>
 </segment>
 </net>
@@
 </segment>
 <segment>
-<pinref part="J1" gate="G$1" pin="4"/>
 <wire x1="33.02" y1="78.74" x2="40.64" y2="78.74" width="0.1524" layer="91"/>
 <label x="40.64" y="78.74" size="0.8128" layer="95" xref="yes"/>
-</segment>
-<segment>
-<pinref part="JP1" gate="A" pin="3"/>
+<pinref part="U$9" gate="G$1" pin="MOSI"/>
+</segment>
+<segment>
+<pinref part="U$6" gate="G$1" pin="4"/>
 <wire x1="-15.24" y1="144.78" x2="0" y2="144.78" width="0.1524" layer="91"/>
 <label x="0" y="144.78" size="1.016" layer="95" xref="yes"/>
@@
 <net name="RESET" class="0">
 <segment>
-<pinref part="J1" gate="G$1" pin="5"/>
-<wire x1="15.24" y1="76.2" x2="10.16" y2="76.2" width="0.1524" layer="91"/>
-<label x="10.16" y="76.2" size="0.8128" layer="95" rot="R180" xref="yes"/>
-</segment>
-<segment>
 <pinref part="U$1" gate="G$1" pin="PC6"/>
 <wire x1="53.34" y1="162.56" x2="53.34" y2="167.64" width="0.1524" layer="91"/>
@@
 </segment>
 <segment>
-<pinref part="JP1" gate="A" pin="5"/>
+<wire x1="149.86" y1="127" x2="134.62" y2="127" width="0.1524" layer="91"/>
+<label x="134.62" y="127" size="1.016" layer="95" rot="R180" xref="yes"/>
+<pinref part="U$7" gate="G$1" pin="2"/>
+</segment>
+<segment>
+<pinref part="U$6" gate="G$1" pin="2"/>
 <wire x1="-15.24" y1="139.7" x2="0" y2="139.7" width="0.1524" layer="91"/>
 <label x="0" y="139.7" size="1.016" layer="95" xref="yes"/>
 </segment>
 <segment>
-<pinref part="JP2" gate="A" pin="5"/>
-<wire x1="149.86" y1="127" x2="134.62" y2="127" width="0.1524" layer="91"/>
-<label x="134.62" y="127" size="1.016" layer="95" rot="R180" xref="yes"/>
+<pinref part="U$9" gate="G$1" pin="RESET"/>
+<wire x1="10.16" y1="76.2" x2="2.54" y2="76.2" width="0.1524" layer="91"/>
+<label x="2.54" y="76.2" size="1.016" layer="95" rot="R180" xref="yes"/>
 </segment>
 </net>
@@
 </segment>
 <segment>
-<pinref part="JP1" gate="A" pin="4"/>
+<wire x1="149.86" y1="129.54" x2="134.62" y2="129.54" width="0.1524" layer="91"/>
+<label x="134.62" y="129.54" size="1.016" layer="95" rot="R180" xref="yes"/>
+<pinref part="U$7" gate="G$1" pin="3"/>
+</segment>
+<segment>
+<pinref part="U$6" gate="G$1" pin="3"/>
 <wire x1="-15.24" y1="142.24" x2="0" y2="142.24" width="0.1524" layer="91"/>
 <label x="0" y="142.24" size="1.016" layer="95" xref="yes"/>
 </segment>
-<segment>
-<pinref part="JP2" gate="A" pin="4"/>
-<wire x1="149.86" y1="129.54" x2="134.62" y2="129.54" width="0.1524" layer="91"/>
-<label x="134.62" y="129.54" size="1.016" layer="95" rot="R180" xref="yes"/>
-</segment>
-</net>
+</net>

Commit message: Added bypass cap and removed deprecated seperate resistor design
Parts:
- added C1: 1uF, resistor:C-USC0603
Connections:
- net GND: now also C1.2
- net VCC: now also C1.1
Changed lines of the file:
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@@
 <part name="U$7" library="ScottSilver" deviceset="DIP1X6MALE" device=""/>
 <part name="U$9" library="ScottSilver" deviceset="DIP2X3MALE" device=""/>
+<part name="C1" library="resistor" deviceset="C-US" device="C0603" value="1uF"/>
+<part name="SUPPLY7" library="SparkFun-Aesthetics" deviceset="VCC" device=""/>
+<part name="GND7" library="SparkFun-Aesthetics" deviceset="GND" device=""/>
 </parts>
 <sheets>
@@
 <instance part="U$7" gate="G$1" x="149.86" y="129.54"/>
 <instance part="U$9" gate="G$1" x="17.78" y="78.74"/>
+<instance part="C1" gate="G$1" x="-30.48" y="144.78"/>
+<instance part="SUPPLY7" gate="G$1" x="-30.48" y="152.4"/>
+<instance part="GND7" gate="1" x="-30.48" y="132.08"/>
 </instances>
 <busses>
@@
 <pinref part="U$7" gate="G$1" pin="6"/>
 </segment>
+<segment>
+<pinref part="C1" gate="G$1" pin="1"/>
+<pinref part="SUPPLY7" gate="G$1" pin="VCC"/>
+<wire x1="-30.48" y1="152.4" x2="-30.48" y2="147.32" width="0.1524" layer="91"/>
+</segment>
 </net>
 <net name="GND" class="0">
@@
 <wire x1="-15.24" y1="137.16" x2="-10.16" y2="137.16" width="0.1524" layer="91"/>
 </segment>
+<segment>
+<pinref part="C1" gate="G$1" pin="2"/>
+<pinref part="GND7" gate="1" pin="GND"/>
+<wire x1="-30.48" y1="134.62" x2="-30.48" y2="139.7" width="0.1524" layer="91"/>
+</segment>
 </net>
