File: LEDMATRIX_SMT_Transistors/Linkable_LED_Matrix.brd (EAGLE design)
At the start: 32 x 32 mm, 9 parts

Commit message: Added Design with Separate Transistors
Parts:
- removed U$2: ULN2803AFWG, ScottSilver:ULN2803AFWG
- added T1, T10, T11, T12, T13, T14, T15, T16, T2, T3, T4, T5, T6, T7, T8, T9: (no value), transistor:SOT23-BEC
- moved U$5 4.18 mm to (7.30, 21.7), flipped to the top
- moved U$1 1.84 mm to (11.5, 17.4)
Connections:
- removed net N$2: U$2.O2, U$3.COL1
- new net N$20: T2.C, U$3.COL1
- new net N$25: T9.C, U$3.ROW7
- new net N$26: T10.C, U$3.ROW6
- new net N$27: T11.C, U$3.ROW5
- new net N$28: T12.C, U$3.ROW4
- new net N$29: T13.C, U$3.ROW3
- new net N$30: T14.C, U$3.ROW2
- new net N$31: T15.C, U$3.ROW1
- new net N$32: T16.C, U$3.ROW0
- net COL0: now also T1.B; no longer U$2.I1
- net COL1: now also T2.B; no longer U$2.I2
- net COL2: now also T3.B; no longer U$2.I3
- net COL3: now also T4.B; no longer U$2.I4
- net COL4: now also T5.B; no longer U$2.I5
- net COL5: now also T6.B; no longer U$2.I6
- net COL6: now also T7.B; no longer U$2.I7
- net COL7: now also T8.B; no longer U$2.I8
- net GND: now also T1.E, T2.E, T3.E, T4.E, T5.E, T6.E, T7.E, T8.E; no longer U$2.GND
- net N$1: now also T1.C; no longer U$2.O1
- net N$3: now also T3.C; no longer U$2.O3
- net N$4: now also T4.C; no longer U$2.O4
- net N$5: now also T5.C; no longer U$2.O5
- net N$6: now also T6.C; no longer U$2.O6
- net N$7: now also T7.C; no longer U$2.O7
- net N$8: now also T8.C; no longer U$2.O8
- net ROW0: now also T16.B; no longer U$3.ROW0
- net ROW1: now also T15.B; no longer U$3.ROW1
- net ROW2: now also T14.B; no longer U$3.ROW2
- net ROW3: now also T13.B; no longer U$3.ROW3
- net ROW4: now also T12.B; no longer U$3.ROW4
- net ROW5: now also T11.B; no longer U$3.ROW5
- net ROW6: now also T10.B; no longer U$3.ROW6
- net ROW7: now also T9.B; no longer U$3.ROW7
- net VCC: now also T10.E, T11.E, T12.E, T13.E, T14.E, T15.E, T16.E, T9.E; no longer U$2.COMMON
Routing:
- net ROW2: track 49.3 -> 8.43 mm, vias 2 -> 1
- net N$8: track 43.0 -> 3.71 mm, vias 1 -> 0
- net COL6: track 5.41 -> 43.0 mm, vias 1 -> 2
- net VCC: track 110.5 -> 145.7 mm, vias 0 -> 6
- net COL3: track 45.9 -> 15.3 mm, vias 3 -> 2
- net GND: track 125.5 -> 155.5 mm, vias 5 -> 2
- net ROW4: track 16.1 -> 43.3 mm, vias 0 -> 3
- net COL1: track 45.0 -> 19.3 mm, vias 3 -> 2
- net COL4: track 7.57 -> 31.9 mm, vias 1 -> 4
- net N$2: track 23.3 -> 0.00 mm
- net N$1: track 25.4 -> 3.34 mm, vias 1 -> 0
- net N$3: track 23.6 -> 5.25 mm
- net MISO: track 53.3 -> 35.7 mm
- net N$5: track 22.6 -> 5.16 mm
- net COL7: track 5.57 -> 20.7 mm, vias 1 -> 2
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Other:
- board text removed: "R2"
- board text removed: "U2"
