File: Accel/PCB/AccelBreakout.sch (EAGLE design)
At the start: 10 parts

Commit message: accel - size, layout, labels
Adjusted size to be 0.6" DIP spacing.  Better orientation and position of all
labels.  Completely rerouted to remove all vias.
Parts:
- renumbered U$23 to U1
Connections:
- net SCL: now also U$3.2; no longer U$3.3
- net SDA: now also U$3.3; no longer U$3.2
Other:
- moved on the sheet: C4
Changed lines of the file:
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@@
 <?xml version="1.0" encoding="utf-8"?>
 <!DOCTYPE eagle SYSTEM "eagle.dtd">
-<eagle version="7.0.0">
+<eagle version="7.1.0">
 <drawing>
 <settings>
@@
 <setting verticaltext="up"/>
 </settings>
-<grid distance="0.1" unitdist="inch" unit="inch" style="lines" multiple="1" display="no" altdistance="0.01" altunitdist="inch" altunit="inch"/>
+<grid distance="0.1" unitdist="inch" unit="inch" style="lines" multiple="1" display="yes" altdistance="0.01" altunitdist="inch" altunit="inch"/>
 <layers>
 <layer number="1" name="Top" color="4" fill="1" visible="no" active="no"/>
@@
 </classes>
 <parts>
-<part name="U$23" library="ScottSilver" deviceset="MMA8653FCR1" device=""/>
+<part name="U1" library="ScottSilver" deviceset="MMA8653FCR1" device=""/>
 <part name="SUPPLY17" library="SparkFun-Aesthetics" deviceset="VCC" device=""/>
 <part name="C1" library="resistor" deviceset="C-US" device="C0603" value="0.1uF"/>
@@
 </plain>
 <instances>
-<instance part="U$23" gate="G$1" x="68.58" y="50.8"/>
+<instance part="U1" gate="G$1" x="68.58" y="50.8"/>
 <instance part="SUPPLY17" gate="G$1" x="25.4" y="76.2"/>
 <instance part="C1" gate="G$1" x="40.64" y="73.66"/>
@@
 <instance part="C3" gate="G$1" x="35.56" y="43.18"/>
 <instance part="GND25" gate="1" x="35.56" y="35.56"/>
-<instance part="C4" gate="G$1" x="88.9" y="43.18"/>
+<instance part="C4" gate="G$1" x="93.98" y="43.18"/>
 <instance part="SUPPLY18" gate="G$1" x="20.32" y="66.04"/>
 <instance part="SUPPLY19" gate="G$1" x="83.82" y="71.12"/>
 <instance part="SUPPLY20" gate="G$1" x="101.6" y="50.8"/>
-<instance part="GND23" gate="1" x="86.36" y="35.56"/>
+<instance part="GND23" gate="1" x="86.36" y="30.48"/>
 <instance part="R1" gate="G$1" x="20.32" y="60.96" rot="R90"/>
 <instance part="R2" gate="G$1" x="83.82" y="66.04" rot="R90"/>
@@
 <wire x1="40.64" y1="76.2" x2="48.26" y2="76.2" width="0.1524" layer="91"/>
 <wire x1="48.26" y1="76.2" x2="48.26" y2="60.96" width="0.1524" layer="91"/>
-<pinref part="U$23" gate="G$1" pin="VDD"/>
+<pinref part="U1" gate="G$1" pin="VDD"/>
 <wire x1="48.26" y1="60.96" x2="53.34" y2="60.96" width="0.1524" layer="91"/>
 <junction x="40.64" y="76.2"/>
@@
 <segment>
 <pinref part="C4" gate="G$1" pin="1"/>
-<pinref part="U$23" gate="G$1" pin="VDDIO"/>
-<wire x1="83.82" y1="50.8" x2="88.9" y2="50.8" width="0.1524" layer="91"/>
-<wire x1="88.9" y1="50.8" x2="101.6" y2="50.8" width="0.1524" layer="91"/>
-<wire x1="88.9" y1="45.72" x2="88.9" y2="50.8" width="0.1524" layer="91"/>
-<junction x="88.9" y="50.8"/>
+<pinref part="U1" gate="G$1" pin="VDDIO"/>
+<wire x1="83.82" y1="50.8" x2="93.98" y2="50.8" width="0.1524" layer="91"/>
+<wire x1="93.98" y1="50.8" x2="101.6" y2="50.8" width="0.1524" layer="91"/>
+<junction x="93.98" y="50.8"/>
 <pinref part="SUPPLY20" gate="G$1" pin="VCC"/>
+<wire x1="93.98" y1="45.72" x2="93.98" y2="50.8" width="0.1524" layer="91"/>
 </segment>
 <segment>
@@
 </segment>
 <segment>
-<pinref part="U$23" gate="G$1" pin="AGND"/>
-<pinref part="U$23" gate="G$1" pin="GND"/>
-<wire x1="83.82" y1="40.64" x2="83.82" y2="45.72" width="0.1524" layer="91"/>
+<pinref part="U1" gate="G$1" pin="AGND"/>
+<pinref part="U1" gate="G$1" pin="GND"/>
 <pinref part="C4" gate="G$1" pin="2"/>
-<wire x1="88.9" y1="38.1" x2="86.36" y2="38.1" width="0.1524" layer="91"/>
-<wire x1="86.36" y1="38.1" x2="83.82" y2="38.1" width="0.1524" layer="91"/>
-<wire x1="83.82" y1="38.1" x2="83.82" y2="40.64" width="0.1524" layer="91"/>
-<pinref part="U$23" gate="G$1" pin="AAGND"/>
+<pinref part="U1" gate="G$1" pin="AAGND"/>
 <wire x1="83.82" y1="55.88" x2="86.36" y2="55.88" width="0.1524" layer="91"/>
 <wire x1="86.36" y1="55.88" x2="86.36" y2="45.72" width="0.1524" layer="91"/>
-<wire x1="86.36" y1="45.72" x2="83.82" y2="45.72" width="0.1524" layer="91"/>
 <pinref part="GND23" gate="1" pin="GND"/>
-<junction x="86.36" y="38.1"/>
+<label x="86.36" y="38.1" size="1.778" layer="95"/>
+<wire x1="86.36" y1="33.02" x2="86.36" y2="35.56" width="0.1524" layer="91"/>
+<junction x="86.36" y="45.72"/>
+<wire x1="86.36" y1="35.56" x2="86.36" y2="40.64" width="0.1524" layer="91"/>
+<wire x1="86.36" y1="40.64" x2="86.36" y2="45.72" width="0.1524" layer="91"/>
+<wire x1="83.82" y1="40.64" x2="86.36" y2="40.64" width="0.1524" layer="91"/>
+<junction x="86.36" y="40.64"/>
+<wire x1="93.98" y1="38.1" x2="93.98" y2="35.56" width="0.1524" layer="91"/>
+<wire x1="86.36" y1="35.56" x2="93.98" y2="35.56" width="0.1524" layer="91"/>
+<junction x="86.36" y="35.56"/>
+<wire x1="83.82" y1="45.72" x2="86.36" y2="45.72" width="0.1524" layer="91"/>
 </segment>
 <segment>
@@
 <segment>
 <pinref part="C3" gate="G$1" pin="1"/>
-<pinref part="U$23" gate="G$1" pin="BYP"/>
+<pinref part="U1" gate="G$1" pin="BYP"/>
 <wire x1="35.56" y1="45.72" x2="53.34" y2="45.72" width="0.1524" layer="91"/>
 </segment>
@@
 <net name="SDA" class="0">
 <segment>
-<pinref part="U$23" gate="G$1" pin="SDA"/>
+<pinref part="U1" gate="G$1" pin="SDA"/>
 <wire x1="83.82" y1="60.96" x2="88.9" y2="60.96" width="0.1524" layer="91"/>
 <label x="88.9" y="60.96" size="1.778" layer="95" xref="yes"/>
@@
 </segment>
 <segment>
-<label x="0" y="35.56" size="1.016" layer="95" xref="yes"/>
-<wire x1="-17.78" y1="35.56" x2="0" y2="35.56" width="0.1524" layer="91"/>
-<pinref part="U$3" gate="G$1" pin="2"/>
+<pinref part="U$3" gate="G$1" pin="3"/>
+<wire x1="-17.78" y1="33.02" x2="0" y2="33.02" width="0.1524" layer="91"/>
+<label x="0" y="33.02" size="1.016" layer="95" xref="yes"/>
 </segment>
 </net>
 <net name="SCL" class="0">
 <segment>
-<pinref part="U$23" gate="G$1" pin="SCL"/>
+<pinref part="U1" gate="G$1" pin="SCL"/>
 <wire x1="53.34" y1="55.88" x2="20.32" y2="55.88" width="0.1524" layer="91"/>
 <label x="20.32" y="55.88" size="1.778" layer="95" rot="R180" xref="yes"/>
@@
 </segment>
 <segment>
-<label x="0" y="33.02" size="1.016" layer="95" xref="yes"/>
-<wire x1="-17.78" y1="33.02" x2="0" y2="33.02" width="0.1524" layer="91"/>
-<pinref part="U$3" gate="G$1" pin="3"/>
+<pinref part="U$3" gate="G$1" pin="2"/>
+<wire x1="-17.78" y1="35.56" x2="0" y2="35.56" width="0.1524" layer="91"/>
+<label x="0" y="35.56" size="1.016" layer="95" xref="yes"/>
 </segment>
 </net>
 <net name="INT1" class="0">
 <segment>
-<pinref part="U$23" gate="G$1" pin="INT1"/>
+<pinref part="U1" gate="G$1" pin="INT1"/>
 <wire x1="53.34" y1="50.8" x2="35.56" y2="50.8" width="0.1524" layer="91"/>
 <label x="35.56" y="50.8" size="1.778" layer="95" rot="R180" xref="yes"/>
@@
 <net name="INT2" class="0">
 <segment>
-<pinref part="U$23" gate="G$1" pin="INT2"/>
+<pinref part="U1" gate="G$1" pin="INT2"/>
 <wire x1="53.34" y1="40.64" x2="43.18" y2="40.64" width="0.1524" layer="91"/>
 <wire x1="43.18" y1="40.64" x2="43.18" y2="25.4" width="0.1524" layer="91"/>

Commit message: accel - adjusted direction symbol, replaced parts
Some old parts were missing from raspberrystem.lbr.
Parts:
- removed U$2: ACCELDIR, ScottSilver:ACCELDIR
- removed U$3, U$4: DIP1X3MALE, OldScottSilver:DIP1X3MALE
- added J1, J2: (no value), raspberrystem:PINHD-1X3
- U1: device ScottSilver:MMA8653FCR1 -> raspberrystem:MMA8653FCR1
Connections:
- net GND: now also J1.3; no longer U$4.3
- net INT1: now also J1.1; no longer U$4.1
- net INT2: now also J1.2; no longer U$4.2
- net SCL: now also J2.2; no longer U$3.2
- net SDA: now also J2.3; no longer U$3.3
- net VCC: now also J2.1; no longer U$3.1
Changed lines of the file:
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@@
 </classes>
 <parts>
-<part name="U1" library="ScottSilver" deviceset="MMA8653FCR1" device=""/>
+<part name="U1" library="raspberrystem" deviceset="MMA8653FCR1" device=""/>
 <part name="SUPPLY17" library="SparkFun-Aesthetics" deviceset="VCC" device=""/>
 <part name="C1" library="resistor" deviceset="C-US" device="C0603" value="0.1uF"/>
@@
 <part name="SUPPLY1" library="SparkFun-Aesthetics" deviceset="VCC" device=""/>
 <part name="GND1" library="SparkFun-Aesthetics" deviceset="GND" device=""/>
-<part name="U$2" library="ScottSilver" deviceset="ACCELDIR" device=""/>
-<part name="U$3" library="OldScottSilver" deviceset="DIP1X3MALE" device=""/>
-<part name="U$4" library="OldScottSilver" deviceset="DIP1X3MALE" device=""/>
+<part name="J2" library="raspberrystem" deviceset="PINHD-1X3" device=""/>
+<part name="J1" library="raspberrystem" deviceset="PINHD-1X3" device=""/>
 </parts>
 <sheets>
@@
 <instance part="SUPPLY1" gate="G$1" x="0" y="38.1"/>
 <instance part="GND1" gate="1" x="0" y="17.78"/>
-<instance part="U$2" gate="G$1" x="81.28" y="20.32"/>
-<instance part="U$3" gate="G$1" x="-17.78" y="35.56"/>
-<instance part="U$4" gate="G$1" x="-17.78" y="22.86"/>
+<instance part="J2" gate="A" x="-17.78" y="35.56"/>
+<instance part="J1" gate="A" x="-17.78" y="22.86"/>
 </instances>
 <busses>
@@
 <segment>
 <pinref part="SUPPLY1" gate="G$1" pin="VCC"/>
-<wire x1="-17.78" y1="38.1" x2="0" y2="38.1" width="0.1524" layer="91"/>
-<pinref part="U$3" gate="G$1" pin="1"/>
+<wire x1="-20.32" y1="38.1" x2="0" y2="38.1" width="0.1524" layer="91"/>
+<pinref part="J2" gate="A" pin="1"/>
 </segment>
 </net>
@@
 <segment>
 <pinref part="GND1" gate="1" pin="GND"/>
-<wire x1="0" y1="20.32" x2="-17.78" y2="20.32" width="0.1524" layer="91"/>
-<pinref part="U$4" gate="G$1" pin="3"/>
+<wire x1="0" y1="20.32" x2="-20.32" y2="20.32" width="0.1524" layer="91"/>
+<pinref part="J1" gate="A" pin="3"/>
 </segment>
 </net>
@@
 </segment>
 <segment>
-<pinref part="U$3" gate="G$1" pin="3"/>
-<wire x1="-17.78" y1="33.02" x2="0" y2="33.02" width="0.1524" layer="91"/>
+<pinref part="J2" gate="A" pin="3"/>
+<wire x1="-20.32" y1="33.02" x2="0" y2="33.02" width="0.1524" layer="91"/>
 <label x="0" y="33.02" size="1.016" layer="95" xref="yes"/>
 </segment>
@@
 </segment>
 <segment>
-<pinref part="U$3" gate="G$1" pin="2"/>
-<wire x1="-17.78" y1="35.56" x2="0" y2="35.56" width="0.1524" layer="91"/>
+<pinref part="J2" gate="A" pin="2"/>
+<wire x1="-20.32" y1="35.56" x2="0" y2="35.56" width="0.1524" layer="91"/>
 <label x="0" y="35.56" size="1.016" layer="95" xref="yes"/>
 </segment>
@@
 <segment>
 <label x="0" y="25.4" size="1.016" layer="95" xref="yes"/>
-<wire x1="-17.78" y1="25.4" x2="0" y2="25.4" width="0.1524" layer="91"/>
-<pinref part="U$4" gate="G$1" pin="1"/>
+<wire x1="-20.32" y1="25.4" x2="0" y2="25.4" width="0.1524" layer="91"/>
+<pinref part="J1" gate="A" pin="1"/>
 </segment>
 </net>
@@
 <segment>
 <label x="0" y="22.86" size="1.016" layer="95" xref="yes"/>
-<wire x1="-17.78" y1="22.86" x2="0" y2="22.86" width="0.1524" layer="91"/>
-<pinref part="U$4" gate="G$1" pin="2"/>
+<wire x1="-20.32" y1="22.86" x2="0" y2="22.86" width="0.1524" layer="91"/>
+<pinref part="J1" gate="A" pin="2"/>
 </segment>
 </net>

Commit message: accel - Moved parts to local library (from raspberrystem.lbr)
Parts:
- J1, J2: device raspberrystem:PINHD-1X3 -> AccelBreakout:PINHD-1X3
- U1: device raspberrystem:MMA8653FCR1 -> AccelBreakout:MMA8653FCR1
Changed lines of the file:
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@@
 <layer number="56" name="wert" color="7" fill="1" visible="no" active="no"/>
 <layer number="57" name="tCAD" color="7" fill="1" visible="no" active="no"/>
+<layer number="90" name="Modules" color="5" fill="1" visible="yes" active="yes"/>
 <layer number="91" name="Nets" color="2" fill="1" visible="yes" active="yes"/>
 <layer number="92" name="Busses" color="1" fill="1" visible="yes" active="yes"/>
@@
 </classes>
 <parts>
-<part name="U1" library="raspberrystem" deviceset="MMA8653FCR1" device=""/>
+<part name="U1" library="AccelBreakout" deviceset="MMA8653FCR1" device=""/>
 <part name="SUPPLY17" library="SparkFun-Aesthetics" deviceset="VCC" device=""/>
 <part name="C1" library="resistor" deviceset="C-US" device="C0603" value="0.1uF"/>
@@
 <part name="SUPPLY1" library="SparkFun-Aesthetics" deviceset="VCC" device=""/>
 <part name="GND1" library="SparkFun-Aesthetics" deviceset="GND" device=""/>
-<part name="J2" library="raspberrystem" deviceset="PINHD-1X3" device=""/>
-<part name="J1" library="raspberrystem" deviceset="PINHD-1X3" device=""/>
+<part name="J2" library="AccelBreakout" deviceset="PINHD-1X3" device=""/>
+<part name="J1" library="AccelBreakout" deviceset="PINHD-1X3" device=""/>
 </parts>
 <sheets>

Commit message: accel - silkscreen and board size changes
Box around R/Cs.  Increased board size to fit better pin labels
Parts:
- C1, C2, C3, C4: device resistor:C-USC0603 -> AccelBreakout:C-USC0603
- R1, R2: device resistor:R-US_R0603 -> AccelBreakout:R-US_R0603
Changed lines of the file:
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@@
 <part name="U1" library="AccelBreakout" deviceset="MMA8653FCR1" device=""/>
 <part name="SUPPLY17" library="SparkFun-Aesthetics" deviceset="VCC" device=""/>
-<part name="C1" library="resistor" deviceset="C-US" device="C0603" value="0.1uF"/>
-<part name="C2" library="resistor" deviceset="C-US" device="C0603" value="1uF"/>
+<part name="C1" library="AccelBreakout" deviceset="C-US" device="C0603" value="0.1uF"/>
+<part name="C2" library="AccelBreakout" deviceset="C-US" device="C0603" value="1uF"/>
 <part name="GND24" library="SparkFun-Aesthetics" deviceset="GND" device=""/>
-<part name="C3" library="resistor" deviceset="C-US" device="C0603" value="0.1uF"/>
+<part name="C3" library="AccelBreakout" deviceset="C-US" device="C0603" value="0.1uF"/>
 <part name="GND25" library="SparkFun-Aesthetics" deviceset="GND" device=""/>
-<part name="C4" library="resistor" deviceset="C-US" device="C0603" value="0.1uF"/>
+<part name="C4" library="AccelBreakout" deviceset="C-US" device="C0603" value="0.1uF"/>
 <part name="SUPPLY18" library="SparkFun-Aesthetics" deviceset="VCC" device=""/>
 <part name="SUPPLY19" library="SparkFun-Aesthetics" deviceset="VCC" device=""/>
 <part name="SUPPLY20" library="SparkFun-Aesthetics" deviceset="VCC" device=""/>
 <part name="GND23" library="SparkFun-Aesthetics" deviceset="GND" device=""/>
-<part name="R1" library="resistor" deviceset="R-US_" device="R0603" value="10K"/>
-<part name="R2" library="resistor" deviceset="R-US_" device="R0603" value="10K"/>
+<part name="R1" library="AccelBreakout" deviceset="R-US_" device="R0603" value="10K"/>
+<part name="R2" library="AccelBreakout" deviceset="R-US_" device="R0603" value="10K"/>
 <part name="SUPPLY1" library="SparkFun-Aesthetics" deviceset="VCC" device=""/>
 <part name="GND1" library="SparkFun-Aesthetics" deviceset="GND" device=""/>
